File: Burnwing.kicad_pcb (KiCad board)
At the start: 2 copper layers, 50.8 x 22.9 mm, 58 parts, among them J1 Conn_01x06_MountingPin, Q1 AONR21307, U1 NCV8402ADDR2G, X1 USB Type C, X3 HUSB238

Commit message: Routing updates
Parts:
- added R3: 0, R_0603_1608Metric_Pad0.98x0.95mm_HandSolder, F.Cu at (80.4, 85.7)
- added R5: 0, R_0603_1608Metric_Pad0.98x0.95mm_HandSolder, F.Cu at (80.4, 97.2)
- added REF**: PinHeader_1x02_P1.00mm_Vertical, Connector_PinHeader_1.00mm:PinHeader_1x02_P1.00mm_Vertical, F.Cu at (85.2, 96.6)
- 12V, 15V, 18V, 9V: footprint Adafruit HUSB238 USB-C PD Breakout:SOLDERJUMPER_ARROW_NOPASTE -> SOLDERJUMPER_ARROW_NOPASTE
- 1A: renamed from SJ6; footprint Adafruit HUSB238 USB-C PD Breakout:SOLDERJUMPER_CLOSEDWIRE -> SOLDERJUMPER_CLOSEDWIRE
- 2A: renamed from SJ7; footprint Adafruit HUSB238 USB-C PD Breakout:SOLDERJUMPER_ARROW_NOPASTE -> SOLDERJUMPER_ARROW_NOPASTE
- 5V: footprint Adafruit HUSB238 USB-C PD Breakout:SOLDERJUMPER_CLOSEDWIRE -> SOLDERJUMPER_CLOSEDWIRE
- Burn1, Burn2: footprint 00-footprint-lib:SW-SMD_4P-L5.1-W5.1-P3.70-LS6.5-TL-2 -> SW-SMD_4P-L5.1-W5.1-P3.70-LS6.5-TL-2
- C1, C2, C3, C4: footprint Adafruit HUSB238 USB-C PD Breakout:0805-NO -> 0805-NO
- D1, D2, D6: footprint LED_SMD:LED_0805_2012Metric -> LED_0805_2012Metric
- G***: footprint Library:LOGO -> LOGO
- H2: footprint MountingHole:MountingHole_2.2mm_M2_Pad -> MountingHole_2.2mm_M2_Pad
- J1: footprint Connector_Molex:Molex_PicoBlade_53261-0671_1x06-1MP_P1.25mm_Horizontal -> Molex_PicoBlade_53261-0671_1x06-1MP_P1.25mm_Horizontal
- PLABEL0: footprint Adafruit HUSB238 USB-C PD Breakout:PLABEL0 -> PLABEL0
- PLABEL10: footprint Adafruit HUSB238 USB-C PD Breakout:PLABEL10 -> PLABEL10
- PLABEL11: footprint Adafruit HUSB238 USB-C PD Breakout:PLABEL11 -> PLABEL11
- PLABEL14: footprint Adafruit HUSB238 USB-C PD Breakout:PLABEL14 -> PLABEL14
- PLABEL16: footprint Adafruit HUSB238 USB-C PD Breakout:PLABEL16 -> PLABEL16
- PLABEL17: footprint Adafruit HUSB238 USB-C PD Breakout:PLABEL17 -> PLABEL17
- PLABEL18: footprint Adafruit HUSB238 USB-C PD Breakout:PLABEL18 -> PLABEL18
- PLABEL3: footprint Adafruit HUSB238 USB-C PD Breakout:PLABEL3 -> PLABEL3
- PLABEL4: footprint Adafruit HUSB238 USB-C PD Breakout:PLABEL4 -> PLABEL4
- PLABEL5: footprint Adafruit HUSB238 USB-C PD Breakout:PLABEL5 -> PLABEL5
- PLABEL6: footprint Adafruit HUSB238 USB-C PD Breakout:PLABEL6 -> PLABEL6
- PLABEL7: footprint Adafruit HUSB238 USB-C PD Breakout:PLABEL7 -> PLABEL7
- PLABEL8: footprint Adafruit HUSB238 USB-C PD Breakout:PLABEL8 -> PLABEL8
- PLABEL9: footprint Adafruit HUSB238 USB-C PD Breakout:PLABEL9 -> PLABEL9
- Q1: footprint Adafruit HUSB238 USB-C PD Breakout:POWERDI3333 -> POWERDI3333
- R1: footprint 00-footprint-lib:AxialBurnResistor -> AxialBurnResistor
- R10: renamed from R7; footprint Adafruit HUSB238 USB-C PD Breakout:0603-NO -> 0603-NO
- R15: value 6K -> 750; footprint Resistor_SMD:R_0603_1608Metric_Pad0.98x0.95mm_HandSolder -> R_0603_1608Metric_Pad0.98x0.95mm_HandSolder
- R16, R17: value 150 -> 510; footprint Adafruit HUSB238 USB-C PD Breakout:0603-NO -> 0603-NO
- R2: footprint 00-footprint-lib:AxialBurnResistor_No_Cutout -> AxialBurnResistor_No_Cutout
- R3, R4, R5, R8: footprint Adafruit HUSB238 USB-C PD Breakout:0603-NO -> 0603-NO
- R7: renamed from R1; footprint Adafruit HUSB238 USB-C PD Breakout:0603-NO -> 0603-NO
- R8: renamed from R2; footprint Adafruit HUSB238 USB-C PD Breakout:0603-NO -> 0603-NO
- R9: renamed from R6; footprint Adafruit HUSB238 USB-C PD Breakout:0603-NO -> 0603-NO
- REF** (x2): footprint Resistor_SMD:R_2512_6332Metric_Pad1.40x3.35mm_HandSolder -> R_2512_6332Metric_Pad1.40x3.35mm_HandSolder
- U1: footprint NCV8402ADDR2G:SOIC8_ONS -> SOIC8_ONS
- X1: footprint Adafruit HUSB238 USB-C PD Breakout:USB_C_CUSB31-CFM2AX-01-X -> USB_C_CUSB31-CFM2AX-01-X
- X3: footprint Adafruit HUSB238 USB-C PD Breakout:DFN10_3X3MM -> DFN10_3X3MM
- p: footprint Connector_Molex:Molex_Pico-Lock_504050-0691_1x06-1MP_P1.50mm_Horizontal -> Molex_Pico-Lock_504050-0691_1x06-1MP_P1.50mm_Horizontal
- moved 2A 0.99 mm to (84.0, 100.7)
- moved R8 0.80 mm to (86.2, 100.7)
- moved 1A 0.72 mm to (88.5, 100.7)
- moved R9 0.63 mm to (87.9, 86.0)
- moved R10 0.52 mm to (85.8, 86.1)
- moved R8 0.49 mm to (89.8, 86.0)
- moved R7 0.30 mm to (91.5, 86.0)
- moved R6 0.25 mm to (125.7, 96.9)
- moved R4 0.25 mm to (125.7, 86.1)
- moved R16 0.19 mm to (103.6, 91.3), turned to 90 degrees
- moved D1 0.18 mm to (105.5, 91.2), turned to 90 degrees
- moved D2 0.11 mm to (107.7, 91.2), turned to 90 degrees
- moved Burn2 0.08 mm to (99.8, 95.6)
- turned PLABEL4 to 180 degrees
Connections:
- Burn1 pad 3: BURN_CTRL_1 -> /GATE1
- Burn2 pad 4: BURN_CTRL_2 -> (no net)
- D1 pad 1: (no net) -> /GATE1
- D1 pad 2: (no net) -> BURN_CTRL_1
- D2 pad 1: (no net) -> /GATE2
- D2 pad 2: (no net) -> BURN_CTRL_2
- D6 pad 1: Net-(X3-VIN) -> GND
- R15 pad 1: Net-(R11-Pad1) -> VOUT
- R15 pad 2: Net-(X3-VSET) -> (no net)
- R16 pad 1: (no net) -> BURN_CTRL_1
- R16 pad 2: (no net) -> BURN_CTRL_1
- R17 pad 1: (no net) -> BURN_CTRL_2
- R17 pad 2: (no net) -> BURN_CTRL_2
Routing:
- net BURN_CTRL_2: track 1.74 -> 23.5 mm
- net BURN_CTRL_1: track 1.84 -> 19.1 mm, vias 0 -> 2
- net VOUT: track 52.0 -> 64.8 mm
- net /GATE2: track 0.00 -> 8.56 mm
- net /GATE1: track 0.00 -> 5.78 mm
- net Net-(H3-Pad1): track 0.00 -> 3.46 mm
- net SCL: track 0.10 -> 2.63 mm
- net (no net): track 0.00 -> 2.40 mm
- net Net-(H1-Pad1): track 0.00 -> 2.34 mm
- net N$10: track 0.00 -> 2.21 mm
- net GND: track 18.7 -> 16.7 mm, vias 32 -> 42
- net N$9: track 4.72 -> 6.12 mm
- net SDA: track 0.00 -> 1.37 mm
- net N$1: track 4.04 -> 3.21 mm
- net VBUS: track 21.5 -> 22.2 mm
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
Commit message: Minor updates
Parts:
- moved R3 0.68 mm to (81.0, 85.9)
- moved R15 0.63 mm to (116.8, 82.3)
- moved R5 0.62 mm to (81.0, 97.1)
- moved D6 0.15 mm to (120.3, 82.4)
- moved C2 0.10 mm to (96.2, 86.2)
- moved C3 0.10 mm to (96.2, 84.2)
- moved C4 0.10 mm to (96.2, 82.1)
Connections:
- Burn1 pad 1: VOUT -> (no net)
- Burn1 pad 3: /GATE1 -> (no net)
- Burn2 pad 1: VOUT -> (no net)
- D6 pad 2: (no net) -> VOUT
- R15 pad 2: (no net) -> VOUT
Routing:
- net BURN_CTRL_2: track 23.5 -> 20.9 mm
- net (no net): track 2.40 -> 0.00 mm
- net VOUT: track 64.8 -> 66.1 mm
- net BURN_CTRL_1: track 19.1 -> 20.1 mm
- net Net-(H1-Pad1): track 2.34 -> 3.27 mm
- net Net-(H3-Pad1): track 3.46 -> 4.18 mm
- net GND: vias 42 -> 45

Commit message: Cleaned up Schematic and exported project libraries
Parts:
- .space: renamed from G***; footprint LOGO -> Library:LOGO
- 12V, 15V, 18V, 2A, 9V: footprint SOLDERJUMPER_ARROW_NOPASTE -> Library:SOLDERJUMPER_ARROW_NOPASTE
- 1A, 5V: footprint SOLDERJUMPER_CLOSEDWIRE -> Library:SOLDERJUMPER_CLOSEDWIRE
- Burn1, Burn2: footprint SW-SMD_4P-L5.1-W5.1-P3.70-LS6.5-TL-2 -> Library:SW-SMD_4P-L5.1-W5.1-P3.70-LS6.5-TL-2
- C1, C2, C3, C4: footprint 0805-NO -> Library:0805-NO
- D1, D2, D6: footprint LED_0805_2012Metric -> Library:LED_0805_2012Metric
- H1, H3, H4: footprint MountingHole:MountingHole_2.2mm_M2_Pad -> Library:MountingHole_2.2mm_M2_Pad
- H2: footprint MountingHole_2.2mm_M2_Pad -> Library:MountingHole_2.2mm_M2_Pad
- J1: footprint Molex_PicoBlade_53261-0671_1x06-1MP_P1.25mm_Horizontal -> Library:Molex_PicoBlade_53261-0671_1x06-1MP_P1.25mm_Horizontal
- J2: renamed from REF**; footprint Connector_PinHeader_1.00mm:PinHeader_1x02_P1.00mm_Vertical -> Library:PinHeader_1x02_P1.00mm_Vertical
- PLABEL0: footprint PLABEL0 -> Library:PLABEL0
- PLABEL10: footprint PLABEL10 -> Library:PLABEL10
- PLABEL11: footprint PLABEL11 -> Library:PLABEL11
- PLABEL14: footprint PLABEL14 -> Library:PLABEL14
- PLABEL16: footprint PLABEL16 -> Library:PLABEL16
- PLABEL17: footprint PLABEL17 -> Library:PLABEL17
- PLABEL18: footprint PLABEL18 -> Library:PLABEL18
- PLABEL3: footprint PLABEL3 -> Library:PLABEL3
- PLABEL4: footprint PLABEL4 -> Library:PLABEL4
- PLABEL5: footprint PLABEL5 -> Library:PLABEL5
- PLABEL6: footprint PLABEL6 -> Library:PLABEL6
- PLABEL7: footprint PLABEL7 -> Library:PLABEL7
- PLABEL8: footprint PLABEL8 -> Library:PLABEL8
- PLABEL9: footprint PLABEL9 -> Library:PLABEL9
- Q1: footprint POWERDI3333 -> Library:POWERDI3333
- R1: footprint AxialBurnResistor -> Library:AxialBurnResistor
- R10, R16, R17, R3, R4, R5, R7, R8, R9: footprint 0603-NO -> Library:0603-NO
- R11: renamed from R3; footprint R_0603_1608Metric_Pad0.98x0.95mm_HandSolder -> Library:R_0603_1608Metric_Pad0.98x0.95mm_HandSolder
- R12: renamed from R4; footprint Resistor_SMD:R_0603_1608Metric_Pad0.98x0.95mm_HandSolder -> Library:R_0603_1608Metric_Pad0.98x0.95mm_HandSolder
- R13: renamed from R5; footprint R_0603_1608Metric_Pad0.98x0.95mm_HandSolder -> Library:R_0603_1608Metric_Pad0.98x0.95mm_HandSolder
- R14: renamed from R6; footprint Resistor_SMD:R_0603_1608Metric_Pad0.98x0.95mm_HandSolder -> Library:R_0603_1608Metric_Pad0.98x0.95mm_HandSolder
- R15: footprint R_0603_1608Metric_Pad0.98x0.95mm_HandSolder -> Library:R_0603_1608Metric_Pad0.98x0.95mm_HandSolder
- R18: renamed from R8; footprint 0603-NO -> Library:0603-NO
- R2: footprint AxialBurnResistor_No_Cutout -> Library:AxialBurnResistor_No_Cutout
- REF** (x2): footprint R_2512_6332Metric_Pad1.40x3.35mm_HandSolder -> Library:R_2512_6332Metric_Pad1.40x3.35mm_HandSolder
- U1: footprint SOIC8_ONS -> Library:SOIC8_ONS
- X1: footprint USB_C_CUSB31-CFM2AX-01-X -> Library:USB_C_CUSB31-CFM2AX-01-X
- X2: renamed from X3; footprint DFN10_3X3MM -> Library:DFN10_3X3MM
- p: footprint Molex_Pico-Lock_504050-0691_1x06-1MP_P1.50mm_Horizontal -> Library:Molex_Pico-Lock_504050-0691_1x06-1MP_P1.50mm_Horizontal
- moved J2 2.57 mm to (86.1, 99.0), turned to 90 degrees
- moved .space 1.69 mm to (112.9, 100.9)
- moved R10 1.61 mm to (84.3, 85.5), turned to 0 degrees
- moved R11 1.37 mm to (79.7, 85.7)
- moved R13 1.28 mm to (79.7, 97.2)
- moved 1A 1.24 mm to (89.5, 99.9)
- moved R7 1.01 mm to (92.4, 85.5), turned to 0 degrees
- moved 2A 0.76 mm to (84.0, 99.9)
- moved R9 0.66 mm to (87.5, 85.5), turned to 0 degrees
- moved R18 0.47 mm to (86.7, 100.7), turned to 0 degrees
- moved R8 0.30 mm to (90.0, 86.3)
- moved PLABEL5 0.30 mm to (84.1, 85.3)
- moved PLABEL11 0.30 mm to (87.3, 91.4)
- moved PLABEL6 0.30 mm to (86.5, 85.4)
- moved 12V 0.19 mm to (88.3, 82.9)
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Routing:
- net GND: track 16.7 -> 8.71 mm, vias 45 -> 44
- net N$3: track 23.2 -> 26.9 mm
- net SDA: track 1.37 -> 2.65 mm
- net N$6: track 1.97 -> 2.87 mm
- net N$8: track 2.42 -> 1.71 mm
- net VBUS: track 22.2 -> 21.6 mm
- net N$7: track 2.36 -> 1.78 mm

Commit message: fixed embedded models
Parts:
- renumbered U1 to Q2
Routing:
- net GND: vias 44 -> 45
