File: Burnwing.kicad_pcb (KiCad board)
At the start: 2 copper layers, 50.8 x 22.9 mm, 47 parts, among them J1 USB Type C, J2 Conn_01x06_MountingPin, J2 Molex_Pico-Lock_504050-0691_1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, J3 Conn_01x02_Pin, Q1 NCV8402ADDR2G, Q2 AONR21307, U1 HUSB238

Commit message: Added Decals and Labels
Parts:
- added G***: LOGO, Library:LOGO, B.Cu at (87.2, 98.8)
- G***: moved to B.Cu
- moved .space 0.56 mm to (114.5, 101.3)
- moved .space 0.08 mm to (105.0, 99.4)
Routing:
- net VDC: track 68.3 -> 67.3 mm
- net GND: vias 106 -> 109
Other:
- board text added: "+"
- board text added: "-"
- board text added: "2025-07-21"
- board text added: "B1"
- board text added: "B2"
- board text added: "Burnwing Rev2"
- board text removed: "Burnwing Rev2 2025-07-21"

Commit message: 4 layer v3 template
Parts:
- removed 12V, 2A, 9V: , Library:SOLDERJUMPER_ARROW_NOPASTE
- removed 1A, 5V: , Library:SOLDERJUMPER_CLOSEDWIRE
- removed J3: Conn_01x02_Pin, Library:PinHeader_1x02_P1.00mm_Vertical
- removed Q1: NCV8402ADDR2G, Library:SOIC-8_L4.9-W3.9-P1.27-LS6.0-BL
- removed R10, R9: 750, Library:R_0603_1608Metric_Pad0.98x0.95mm_HandSolder
- removed the R7 at (87.7, 96.2)
- added 12V1: SOLDERJUMPER, Library:SOLDERJUMPER_ARROW_NOPASTE, F.Cu at (70.0, 113.3)
- added 1A1: SOLDERJUMPERCLOSED, Library:SOLDERJUMPER_CLOSEDWIRE, F.Cu at (70.0, 116.6)
- added 2A1: SOLDERJUMPER, Library:SOLDERJUMPER_ARROW_NOPASTE, F.Cu at (70.0, 119.8)
- added 5V1: SOLDERJUMPERCLOSED, Library:SOLDERJUMPER_CLOSEDWIRE, F.Cu at (70.0, 123.0)
- added R18: 14K, Library:R_0603_1608Metric_Pad0.98x0.95mm_HandSolder, F.Cu at (125.7, 117.8)
- added U2: BTS7030-2EPA, EasyEDA:PG-TSDSO-14_L4.9-W3.9-P0.65-LS6.0-BL-EP, F.Cu at (120.4, 115.5)
- Burn1, Burn2: value Tactile_Button -> KEY-SMD_4P-L6.0-W6.0-P4.50-LS9.5-BR; footprint Library:SW-SMD_4P-L5.1-W5.1-P3.70-LS6.5-TL-2 -> EasyEDA:KEY-SMD_4P-L6.0-W6.0-P4.50-LS9.5-BR
- J2: value Molex_Pico-Lock_504050-0691_1x06-1MP_P1.50mm_Horizontal -> Conn_01x06_MountingPin; footprint Library:Molex_Pico-Lock_504050-0691_1x06-1MP_P1.50mm_Horizontal -> Library:Molex_PicoBlade_53261-0671_1x06-1MP_P1.25mm_Horizontal
- R15, R16: value 750 -> 5.1K
- moved R15 32.6 mm to (125.7, 112.8), turned to 0 degrees
- moved R16 32.0 mm to (125.7, 115.3), turned to 0 degrees
- moved Burn2 25.3 mm to (108.7, 121.7), turned to 0 degrees
- moved Burn1 24.6 mm to (95.2, 121.2), turned to 0 degrees
- moved D1 21.7 mm to (98.2, 113.2)
- moved D2 21.1 mm to (105.6, 112.5)
- moved R7 19.9 mm to (83.7, 114.9), turned to 90 degrees
- moved C1 18.4 mm to (95.0, 106.5)
- moved R8 17.7 mm to (88.2, 113.9)
- moved U1 14.5 mm to (89.7, 106.7)
- moved REF** 1.30 mm to (116.8, 91.4)
- moved R2 1.29 mm to (121.9, 91.4)
- moved R4 1.05 mm to (90.3, 86.4), turned to 180 degrees
- moved REF** 0.92 mm to (121.0, 91.4)
- moved R1 0.64 mm to (115.8, 91.4)
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- renumbered R18 to R7
Connections:
- Burn1 pad 1: Net-(Burn1-A) -> VDC
- Burn1 pad 2: Net-(Burn1-A) -> VDC
- Burn2 pad 1: (no net) -> VDC
- Burn2 pad 2: Net-(Burn2-A) -> VDC
- Burn2 pad 3: (no net) -> BURN_CTRL_2
- C2 pad 2: GND -> Net-(C2-Pad2)
- C3 pad 2: GND -> Net-(C2-Pad2)
- C4 pad 2: GND -> Net-(C2-Pad2)
- D1 pad 2: BURN_CTRL_1 -> Net-(D1-A)
- D2 pad 2: BURN_CTRL_2 -> Net-(D2-A)
- J2 pad 1: VDC -> GND (x2)
- J2 pad 2: BURN_CTRL_1 -> VDC (x2)
- J2 pad 3: GND -> BURN_CTRL_1 (x2)
- R1 pad 1: VDC -> GND
- R1 pad 2: Net-(Q1-D1-Pad7) -> Net-(R1-Pad2)
- R15 pad 1: BURN_CTRL_2 -> BURN_CTRL_1
- R15 pad 2: BURN_CTRL_2 -> Net-(D1-A)
- R16 pad 1: BURN_CTRL_1 -> BURN_CTRL_2
- R16 pad 2: BURN_CTRL_1 -> Net-(D2-A)
- R2 pad 1: VDC -> GND
- R2 pad 2: Net-(Q1-D2-Pad5) -> Net-(R2-Pad2)
Routing:
- net VDC: track 67.3 -> 8.17 mm
- net BURN_CTRL_1: track 41.9 -> 0.00 mm
- net Net-(Q1-D2-Pad5): track 24.4 -> 0.00 mm
- net BURN_CTRL_2: track 14.7 -> 0.00 mm
- net Net-(U1-VSET): track 14.3 -> 0.00 mm
- net Net-(Q1-D1-Pad7): track 13.5 -> 0.00 mm
- net Net-(U1-ISET): track 11.1 -> 0.00 mm
- net /D+: track 9.62 -> 0.00 mm
- net Net-(Burn1-A): track 9.37 -> 0.00 mm
- net /D-: track 8.94 -> 0.00 mm, vias 2 -> 0
- net GND: track 9.10 -> 2.72 mm, vias 109 -> 0
- net /CC1: track 5.43 -> 0.00 mm, vias 2 -> 0
- net /CC2: track 3.50 -> 0.00 mm
- net Net-(U1-GATE): track 3.42 -> 0.00 mm
- net Net-(Burn2-A): track 3.34 -> 0.00 mm
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- added copper zone on B.Cu, net (none)
- added copper zone on F.Cu, net (none)
- added copper zone on In2.Cu, net GND
- added copper zone on In1.Cu, net VDC
- removed copper zone on B.Cu, net GND
- removed copper zone on F.Cu, net GND
Other:
- outline, holes or cut-outs redrawn
- copper layers 2 -> 4
- board text removed: "+"
- board text removed: "-"
- board text removed: "B1"
- board text removed: "B2"
