File: Burnwing.kicad_sch (KiCad schematic)
At the start: 57 parts, among them J1 Conn_01x04_Socket, J2 USB Type C, J3 Conn_01x02_Pin, J4 Conn_01x02_Pin, J5 Conn_01x06_MountingPin, J6 Conn_01x06_MountingPin, Q1 AONR21307, SW1 SW_DIP_x02, U1 HUSB238, U2 BTS7030-2EPA, U3 TPS70933QDBVRQ1

Commit message: Fix control-input drive margin, correct LED part, complete BOM
An external controller could not be guaranteed to assert U2 IN0/IN1. The 150R
LED series resistors clamped BURN_CTRL to ~2.05 V, putting the inputs at 1.97 V
against a 2.19 V requirement - V_DI(TH) max 2.0 V plus the GND-network offset
(I_GND 4 mA x R32 47R = 188 mV). Worst case was -220 mV, so the manual buttons
fired a channel while an external controller might not, and only at the hot
corner or on a worst-case part.

Input network:
- R1, R2, R16: 150R -> 1k5. The LED is a clamp, not a load, so the node sits at
  a conductance-weighted average of the rail and Vf. This cuts the LED's
  authority over the control node from 87% to 40% and desensitises it to Vf
  tempco
- R24, R25: 1k -> 330R. Stiffens the pull-up while keeping meaningful series
  protection on a line that leaves the board at J5/J6. Fault current into a
  3.3 V host on a short to VDC is 5.2 mA, against 1.7 mA at 1k and 17 mA at 100R
- R27, R28: populated at 22k, previously DNP at 10k

Result: 2.56 V worst case at 85 C, +367 mV margin (+410 mV at 25 C). Conditions:
3.3 V rail -2%, resistors +/-1%, I_DI(H) 25 uA on the divider Thevenin impedance.

Populating R27/R28 reverses the decision recorded in #5. The parasitic ground
path that motivated leaving them out already exists and is dominated by R23/R26,
the 10k DEN/DSEL pull-downs the driver datasheet requires for unused inputs;
those contribute ~200 uS against ~91 uS for R27/R28 at 22k. 22k rather than the
100k suggested there because 25 uA across 100k is 2.5 V, well above the 0.8 V
guaranteed-low. With them fitted the inputs still sit higher than they did
unpopulated, because the LED clamp was always the dominant term. See #5, #15.

LED part:
- D3, D4, D7: C94868 -> C2286. C94868 is an 0805 part on an 0603 land pattern.
  A previous assembly order was held for exactly this and the corrected part was
  sent by email but never committed, so the mismatch persisted. C2286 (KT-0603R)
  is 0603,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
Parts:
- D3, D4, D7: LCSC C94868 -> C2286
- J5, J6: LCSC (none) -> C563981
- R1, R16, R2: value 150 -> 1k5; LCSC C22808 -> C22843
- R23, R26: LCSC (none) -> C98220
- R24, R25: value 1k -> 330; LCSC (none) -> C23138
- R27, R28: value 10k -> 22k; LCSC (none) -> C31850; now fitted; now in the parts list
- R32: LCSC (none) -> C23182
- SW1: LCSC (none) -> C7430304
Changed lines of the file:
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@@
 		(body_style 1)
 		(exclude_from_sim no)
-		(in_bom no)
+		(in_bom yes)
 		(on_board yes)
-		(in_pos_files no)
-		(dnp yes)
+		(in_pos_files yes)
+		(dnp no)
 		(property "Reference" "R28"
 			(at 190.754 152.4 90)
@@
 			)
 		)
-		(property "Value" "10k"
+		(property "Value" "22k"
 			(at 195.58 152.4 90)
 			(show_name no)
@@
 			)
 		)
+		(property "LCSC" "C31850"
+			(at 0 0 0)
+			(hide yes)
+			(show_name no)
+			(do_not_autoplace no)
+			(effects
+				(font
+					(size 1.27 1.27)
+				)
+			)
+		)
 		(pin "1"
 		)
@@
 			)
 		)
-		(property "Value" "150"
+		(property "Value" "1k5"
 			(at 86.36 105.41 90)
 			(show_name no)
@@
 			)
 		)
-		(property "LCSC" "C22808"
+		(property "LCSC" "C22843"
 			(at 0 0 0)
 			(hide yes)
@@
 			)
 		)
-		(property "Value" "150"
+		(property "Value" "1k5"
 			(at 68.58 105.41 90)
 			(show_name no)
@@
 			)
 		)
-		(property "LCSC" "C22808"
+		(property "LCSC" "C22843"
 			(at 0 0 0)
 			(hide yes)
@@
 		(body_style 1)
 		(exclude_from_sim no)
-		(in_bom no)
+		(in_bom yes)
 		(on_board yes)
-		(in_pos_files no)
-		(dnp yes)
+		(in_pos_files yes)
+		(dnp no)
 		(property "Reference" "R27"
 			(at 183.134 152.4 90)
@@
 			)
 		)
-		(property "Value" "10k"
+		(property "Value" "22k"
 			(at 187.96 152.4 90)
 			(show_name no)
@@
 			)
 		)
+		(property "LCSC" "C31850"
+			(at 0 0 0)
+			(hide yes)
+			(show_name no)
+			(do_not_autoplace no)
+			(effects
+				(font
+					(size 1.27 1.27)
+				)
+			)
+		)
 		(pin "1"
 		)
@@
 		(pin "2"
 		)
-		(instances
+		    (property "LCSC" "C23182"
+      (at 0 0 0)
+      (effects (font (size 1.27 1.27)) (hide yes))
+    )
+    (instances
 			(project "Burnwing"
 				(path "/668c3a07-3236-4b27-b3a6-03c249258f7f"
@@
 			)
 		)
-		(property "LCSC" "C94868"
+		(property "LCSC" "C2286"
 			(at 59.69 114.3 0)
 			(hide yes)
@@
 		(pin "2"
 		)
-		(instances
+		    (property "LCSC" "C563981"
+      (at 0 0 0)
+      (effects (font (size 1.27 1.27)) (hide yes))
+    )
+    (instances
 			(project "Burnwing"
 				(path "/668c3a07-3236-4b27-b3a6-03c249258f7f"
@@
 		(pin "2"
 		)
-		(instances
+		    (property "LCSC" "C98220"
+      (at 0 0 0)
+      (effects (font (size 1.27 1.27)) (hide yes))
+    )
+    (instances
 			(project "Burnwing"
 				(path "/668c3a07-3236-4b27-b3a6-03c249258f7f"
@@
 		(pin "2"
 		)
-		(instances
+		    (property "LCSC" "C98220"
+      (at 0 0 0)
+      (effects (font (size 1.27 1.27)) (hide yes))
+    )
+    (instances
 			(project "Burnwing"
 				(path "/668c3a07-3236-4b27-b3a6-03c249258f7f"
@@
 			)
 		)
-		(property "Value" "1k"
+		(property "Value" "330"
 			(at 82.55 182.88 90)
 			(show_name no)
@@
 			)
 		)
+		(property "LCSC" "C23138"
+			(at 0 0 0)
+			(hide yes)
+			(show_name no)
+			(do_not_autoplace no)
+			(effects
+				(font
+					(size 1.27 1.27)
+				)
+			)
+		)
 		(pin "2"
 		)
@@
 			)
 		)
-		(property "LCSC" "C94868"
+		(property "LCSC" "C2286"
 			(at 71.12 114.3 0)
 			(hide yes)
@@
 		(pin "2"
 		)
-		(instances
+		    (property "LCSC" "C563981"
+      (at 0 0 0)
+      (effects (font (size 1.27 1.27)) (hide yes))
+    )
+    (instances
 			(project "Burnwing"
 				(path "/668c3a07-3236-4b27-b3a6-03c249258f7f"
@@
 			)
 		)
-		(property "Value" "1k"
+		(property "Value" "330"
 			(at 82.55 190.5 90)
 			(show_name no)
@@
 			)
 		)
+		(property "LCSC" "C23138"
+			(at 0 0 0)
+			(hide yes)
+			(show_name no)
+			(do_not_autoplace no)
+			(effects
+				(font
+					(size 1.27 1.27)
+				)
+			)
+		)
 		(pin "2"
 		)
@@
 			)
 		)
-		(property "LCSC" "C94868"
+		(property "LCSC" "C2286"
 			(at 88.9 114.3 0)
 			(hide yes)
@@
 		(pin "3"
 		)
-		(instances
+		    (property "LCSC" "C7430304"
+      (at 0 0 0)
+      (effects (font (size 1.27 1.27)) (hide yes))
+    )
+    (instances
 			(project "Burnwing"
 				(path "/668c3a07-3236-4b27-b3a6-03c249258f7f"
@@
 			)
 		)
-		(property "Value" "150"
+		(property "Value" "1k5"
 			(at 57.15 107.315 90)
 			(show_name no)
@@
 			)
 		)
-		(property "LCSC" "C22808"
+		(property "LCSC" "C22843"
 			(at 0 0 0)
 			(hide yes)
